File: PCB/_restore_backup_2026-08-21T12-02-36-937/Tank_Sensor.kicad_pcb (KiCad board)
At the start: 2 copper layers, 57 x 55 mm, 31 parts, among them J2 SWD_Prog, J3 Sensor_Conn, J4(Tx) Debug_UART, Q1 BC547, Q2 BC547, Q3 BC547, Q4 BC547, Q5 AO3401A, SW1 BTN_6mm, SW2 Power_Switch, U1 CH32V003F4P6, U2 Ai-Thinker-Ra-02

Commit message: update led or mosfet logic or level detect logic
Parts:
- added Q6: AO3401A, Package_TO_SOT_SMD:SOT-23, F.Cu at (80.1, 153.0)
- added R9: 100k, Resistor_SMD:R_0603_1608Metric, F.Cu at (84.5, 152.0)
Routing:
- net GND: track 266.9 -> 265.1 mm
