File: PCB/Tank_Sensor.kicad_pcb (KiCad board)
At the start: 2 copper layers, 57 x 55 mm, 31 parts, among them J2 SWD_Prog, J3 Sensor_Conn, J4(Tx) Debug_UART, Q1 BC547, Q2 BC547, Q3 BC547, Q4 BC547, Q5 AO3401A, SW1 BTN_6mm, SW2 Power_Switch, U1 CH32V003F4P6, U2 Ai-Thinker-Ra-02

Commit message: Hardware Components & BOM List
Routing:
- net /UART_TX: track 35.9 -> 29.3 mm
- net GND: track 266.9 -> 265.1 mm
