File: PCB/Tank_Sensor.kicad_sch (KiCad schematic)
At the start: 35 parts, among them J1 2xAA_Battery, J2 SWD_Prog, J3 Sensor_Conn, J4 Debug_UART, Q1 BC547, Q2 BC547, Q3 BC547, Q4 BC547, Q5 AO3401A, SW1 BTN_6mm, SW2 Power_Switch, U1 CH32V003F4P6, U2 Ai-Thinker-Ra-02

Commit message: Hardware Components & BOM List
Changed lines of the file:
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@@
+	(wire
+		(pts
+			(xy 270.51 186.69) (xy 270 183.81)
+		)
+		(stroke
+			(width 0)
+			(type default)
+		)
+	)
 	(wire
 		(pts
@@
 	(wire
 		(pts
-			(xy 279.4 129.54) (xy 279.4 130.81)
+			(xy 270.51 172.72) (xy 270 176.19)
 		)
 		(stroke
@@
 		)
 	)
+	(wire
+		(pts
+			(xy 279.4 129.54) (xy 279.4 130.81)
+		)
+		(stroke
+			(width 0)
+			(type default)
+		)
+	)
 	(label "SENSOR_POWER_PIN"
 		(at 169.84 122.54 180)
@@
 	)
 	(label "LED_DRIVE"
-		(at 270 176.19 90)
+		(at 270.51 172.72 0)
 		(effects
 			(font
@@
 	)
 	(label "LED_A"
-		(at 270 183.81 90)
-		(effects
-			(font
+		(at 270.51 186.69 0)
+		(effects
+			(font
